Commit message: update

File: assets/robots/xarm6/xarm6_wo_ee_ori_jl.urdf (robot description, URDF)
Before this commit: robot xarm6, 9 links, 8 joints
Links:
- added link eef_point
Joints:
- added joint dummy_eef: type fixed, parent link_eef, child eef_point, origin xyz=-0.06 0.02 0.03 rpy=3.1416 -1.5708 0

Commit message: update

File: assets/robots/xarm6/xarm6_wo_ee_ori_jl.urdf (robot description, URDF)
Before this commit: robot xarm6, 10 links, 9 joints
Joints:
- joint dummy_eef: origin xyz=-0.06 0.02 0.03 rpy=3.1416 -1.5708 0 -> xyz=-0.03 0.02 0.012 rpy=3.1416 -1.5708 0

Commit message: update

File: assets/robots/xarm6/xarm6_wo_ee_ori_jl.urdf (robot description, URDF)
Before this commit: robot xarm6, 10 links, 9 joints
Joints:
- joint dummy_eef: origin xyz=-0.03 0.02 0.012 rpy=3.1416 -1.5708 0 -> xyz=-0.03 0.02 0.02 rpy=3.1416 -1.5708 0
